File: VS_Simple_Circuit.kicad_pcb (KiCad board)
At the start: 2 copper layers, 100 x 50 mm, 7 parts, among them SW1 Button

Commit message: Add PCBWay sponsorship logo
Parts:
- added G***: LOGO, PCBWay-Logo:PCBWay-Logo, F.Cu at (165.1, 58.4)
Other:
- board text added: "Sponsored by:"
- board text added: "pcbway.com"
Changed lines of the file:
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@@
     (area 84.924999 49.924999 185.075001 100.075001)
     (thickness 1.6)
-    (drawings 11)
+    (drawings 13)
     (tracks 18)
     (zones 0)
-    (modules 7)
+    (modules 8)
     (nets 5)
   )
@@
       (xy 28.02891 4.586111) (xy 28.559812 4.875046)) (layer F.Mask) (width 0.01))
   )
+  (module PCBWay-Logo:PCBWay-Logo (layer F.Cu)
+    (at 165.1 58.42)
+    (fp_text reference G*** (at 0 0) (layer B.SilkS) hide
+      (effects (font (thickness 0.3)))
+    )
+    (fp_text value LOGO (at 0.75 0) (layer B.SilkS) hide
+      (effects (font (thickness 0.3)))
+    )
+    (fp_poly (pts (xy -3.830717 2.211349) (xy -1.23409 2.276314) (xy 1.434755 2.391539) (xy 4.062506 2.553975)
+      (xy 6.53585 2.760571) (xy 7.010076 2.807747) (xy 9.318253 3.060664) (xy 11.493435 3.330028)
+      (xy 13.476531 3.606088) (xy 15.208447 3.879093) (xy 16.630091 4.139292) (xy 17.682369 4.376932)
+      (xy 18.306189 4.582263) (xy 18.454845 4.696354) (xy 18.448239 4.879804) (xy 18.231895 4.971342)
+      (xy 17.738837 4.967152) (xy 16.902084 4.863413) (xy 15.654658 4.656309) (xy 14.684375 4.481422)
+      (xy 11.123713 3.894768) (xy 7.352069 3.392614) (xy 3.498482 2.985875) (xy -0.30801 2.685468)
+      (xy -3.938366 2.502308) (xy -7.263547 2.447311) (xy -8.995833 2.478251) (xy -12.832292 2.605734)
+      (xy -10.054167 2.34851) (xy -8.354068 2.244398) (xy -6.241814 2.199694) (xy -3.830717 2.211349)) (layer B.SilkS) (width 0.01))
+    (fp_poly (pts (xy -12.923862 -3.154765) (xy -12.7 -3.107035) (xy -12.790063 -2.847862) (xy -13.031498 -2.20973)
+      (xy -13.381178 -1.305803) (xy -13.586316 -0.781419) (xy -14.078103 0.624283) (xy -14.279899 1.629282)
+      (xy -14.189831 2.276727) (xy -13.806024 2.60977) (xy -13.43613 2.676525) (xy -13.075441 2.722022)
+      (xy -13.224563 2.808894) (xy -13.295313 2.828217) (xy -13.68768 3.046162) (xy -13.758333 3.1944)
+      (xy -13.975222 3.382055) (xy -14.475438 3.436264) (xy -15.033306 3.368268) (xy -15.423149 3.189304)
+      (xy -15.476106 3.108854) (xy -15.609354 2.740061) (xy -15.885418 1.988178) (xy -16.262721 0.966117)
+      (xy -16.658427 -0.102026) (xy -17.078588 -1.242218) (xy -17.421054 -2.186432) (xy -17.649303 -2.832946)
+      (xy -17.727084 -3.078588) (xy -17.497205 -3.147164) (xy -16.957784 -3.175) (xy -16.49027 -3.12545)
+      (xy -16.201055 -2.889625) (xy -15.980589 -2.336767) (xy -15.849431 -1.852084) (xy -15.62394 -1.104952)
+      (xy -15.413858 -0.625286) (xy -15.317078 -0.529167) (xy -15.132813 -0.757861) (xy -14.867676 -1.34493)
+      (xy -14.684375 -1.852083) (xy -14.393088 -2.63249) (xy -14.116188 -3.027359) (xy -13.737164 -3.163877)
+      (xy -13.472486 -3.175) (xy -12.923862 -3.154765)) (layer B.SilkS) (width 0.01))
+    (fp_poly (pts (xy -16.068402 3.00145) (xy -16.059607 3.088309) (xy -16.473801 3.123783) (xy -16.536459 3.12342)
+      (xy -16.946815 3.085268) (xy -16.907644 3.004739) (xy -16.862152 2.991646) (xy -16.285808 2.952912)
+      (xy -16.068402 3.00145)) (layer B.SilkS) (width 0.01))
+    (fp_poly (pts (xy -9.093031 -3.374236) (xy -8.546482 -3.168837) (xy -8.323936 -2.774771) (xy -8.307118 -2.636632)
+      (xy -8.412482 -2.386401) (xy -8.842204 -2.265118) (xy -9.604275 -2.239757) (xy -10.4932 -2.178465)
+      (xy -10.956079 -2.013825) (xy -10.965735 -1.797475) (xy -10.494992 -1.581049) (xy -10.005164 -1.478062)
+      (xy -8.882141 -1.147075) (xy -8.178011 -0.598589) (xy -7.9375 0.122729) (xy -8.15654 0.962087)
+      (xy -8.728306 1.509985) (xy -9.524769 1.696073) (xy -10.384896 1.467486) (xy -10.883602 1.27663)
+      (xy -11.111111 1.32392) (xy -11.1125 1.338607) (xy -11.340888 1.519458) (xy -11.840104 1.588121)
+      (xy -12.567708 1.588743) (xy -12.49666 -0.15434) (xy -11.1125 -0.15434) (xy -10.912015 0.462355)
+      (xy -10.432787 0.763505) (xy -9.858154 0.681219) (xy -9.548264 0.424906) (xy -9.397582 0.034699)
+      (xy -9.667058 -0.368844) (xy -10.261094 -0.754748) (xy -10.779404 -0.755352) (xy -11.082631 -0.391337)
+      (xy -11.1125 -0.15434) (xy -12.49666 -0.15434) (xy -12.481444 -0.527634) (xy -12.37379 -1.817851)
+      (xy -12.128955 -2.668304) (xy -11.676002 -3.164235) (xy -10.94399 -3.390886) (xy -10.061441 -3.435532)
+      (xy -9.093031 -3.374236)) (layer B.SilkS) (width 0.01))
+    (fp_poly (pts (xy -3.633368 -4.976489) (xy -3.212468 -4.90872) (xy -2.927762 -4.732729) (xy -2.710369 -4.338683)
+      (xy -2.491409 -3.616748) (xy -2.297645 -2.846618) (xy -2.0416 -1.911089) (xy -1.805641 -1.23241)
+      (xy -1.630945 -0.923862) (xy -1.597303 -0.919983) (xy -1.461698 -1.221654) (xy -1.281934 -1.90912)
+      (xy -1.09295 -2.844951) (xy -1.059771 -3.034303) (xy -0.877604 -4.041536) (xy -0.718807 -4.635316)
+      (xy -0.523313 -4.924741) (xy -0.231056 -5.018907) (xy 0.037427 -5.027083) (xy 0.410609 -5.00551)
+      (xy 0.644956 -4.889316) (xy 0.740297 -4.601292) (xy 0.696461 -4.064226) (xy 0.513275 -3.200911)
+      (xy 0.190569 -1.934134) (xy 0.029206 -1.322917) (xy -0.706643 1.455208) (xy -2.542993 1.613312)
+      (xy -3.017961 -0.401394) (xy -3.254843 -1.326995) (xy -3.461423 -1.992973) (xy -3.601278 -2.285796)
+      (xy -3.62267 -2.286358) (xy -3.747197 -1.982734) (xy -3.951843 -1.307267) (xy -4.19353 -0.402741)
+      (xy -4.206659 -0.350705) (xy -4.456311 0.593088) (xy -4.667396 1.139348) (xy -4.924732 1.405125)
+      (xy -5.313135 1.507467) (xy -5.5716 1.532958) (xy -6.482292 1.610708) (xy -7.250134 -1.377458)
+      (xy -7.563965 -2.587465) (xy -7.837921 -3.622876) (xy -8.04097 -4.367742) (xy -8.138338 -4.696354)
+      (xy -8.012626 -4.949014) (xy -7.446839 -5.027083) (xy -6.893683 -4.960856) (xy -6.584556 -4.661961)
+      (xy -6.370925 -4.034896) (xy -6.150006 -3.087335) (xy -5.952791 -2.058118) (xy -5.930036 -1.918229)
+      (xy -5.783594 -1.233128) (xy -5.62355 -0.834749) (xy -5.567493 -0.79375) (xy -5.430793 -1.033196)
+      (xy -5.229182 -1.670656) (xy -4.999297 -2.584812) (xy -4.923594 -2.925968) (xy -4.465403 -5.058185)
+      (xy -3.633368 -4.976489)) (layer B.SilkS) (width 0.01))
+    (fp_poly (pts (xy 6.35 1.5875) (xy 4.401306 1.5875) (xy 3.280793 1.555553) (xy 2.528131 1.437791)
+      (xy 1.984661 1.201329) (xy 1.755473 1.03913) (xy 1.169068 0.302297) (xy 1.058333 -0.264888)
+      (xy 1.130443 -0.587005) (xy 2.76238 -0.587005) (xy 2.763402 -0.086066) (xy 3.146595 0.33231)
+      (xy 3.906345 0.527363) (xy 4.001147 0.529167) (xy 4.510008 0.475563) (xy 4.721097 0.209018)
+      (xy 4.7625 -0.413639) (xy 4.726934 -1.037344) (xy 4.526041 -1.278247) (xy 4.018528 -1.282167)
+      (xy 3.929287 -1.273535) (xy 3.149138 -1.029748) (xy 2.76238 -0.587005) (xy 1.130443 -0.587005)
+      (xy 1.222505 -0.998244) (xy 1.627364 -1.589126) (xy 2.141422 -1.850904) (xy 2.176572 -1.852083)
+      (xy 2.244892 -2.01052) (xy 2.025382 -2.335938) (xy 1.663291 -3.032741) (xy 1.654954 -3.219097)
+      (xy 3.175 -3.219097) (xy 3.301662 -2.64739) (xy 3.755874 -2.407134) (xy 4.145139 -2.38125)
+      (xy 4.618372 -2.502057) (xy 4.761211 -2.959996) (xy 4.7625 -3.042709) (xy 4.67707 -3.515434)
+      (xy 4.31392 -3.68837) (xy 3.96875 -3.704167) (xy 3.378249 -3.613744) (xy 3.178382 -3.295809)
+      (xy 3.175 -3.219097) (xy 1.654954 -3.219097) (xy 1.628479 -3.810886) (xy 1.924265 -4.441077)
+      (xy 1.99396 -4.505872) (xy 2.446748 -4.687159) (xy 3.260879 -4.85031) (xy 4.268725 -4.962659)
+      (xy 4.37521 -4.969938) (xy 6.35 -5.096672) (xy 6.35 1.5875)) (layer B.SilkS) (width 0.01))
+    (fp_poly (pts (xy 17.991667 1.5875) (xy 17.330208 1.5875) (xy 16.917291 1.536038) (xy 16.724831 1.285862)
+      (xy 16.670453 0.693286) (xy 16.66875 0.433729) (xy 16.66875 -0.720042) (xy 15.279687 -0.882064)
+      (xy 14.076804 -1.178746) (xy 13.31852 -1.746578) (xy 12.984905 -2.603276) (xy 12.964583 -2.939728)
+      (xy 12.991774 -3.096144) (xy 14.33408 -3.096144) (xy 14.432695 -2.43785) (xy 14.95849 -2.000426)
+      (xy 15.775105 -1.852083) (xy 16.370971 -1.894042) (xy 16.617896 -2.127154) (xy 16.668593 -2.712269)
+      (xy 16.66875 -2.793338) (xy 16.66875 -3.734593) (xy 15.546553 -3.653234) (xy 14.765556 -3.527853)
+      (xy 14.395274 -3.265956) (xy 14.33408 -3.096144) (xy 12.991774 -3.096144) (xy 13.107743 -3.763229)
+      (xy 13.574894 -4.318462) (xy 14.422547 -4.639279) (xy 15.707208 -4.759532) (xy 16.007292 -4.7625)
+      (xy 17.991667 -4.7625) (xy 17.991667 1.5875)) (layer B.SilkS) (width 0.01))
+    (fp_poly (pts (xy 10.708189 -4.426531) (xy 11.711622 -3.790069) (xy 12.399684 -2.834236) (xy 12.573994 -2.329156)
+      (xy 12.589954 -1.326836) (xy 12.253138 -0.265835) (xy 11.648961 0.615879) (xy 11.45454 0.789613)
+      (xy 10.6092 1.184985) (xy 9.528049 1.340206) (xy 8.429086 1.254053) (xy 7.530312 0.925302)
+      (xy 7.371499 0.812531) (xy 6.966252 0.392348) (xy 6.982769 0.075933) (xy 7.062162 -0.018694)
+      (xy 7.393412 -0.18272) (xy 7.911588 -0.070633) (xy 8.325772 0.110476) (xy 9.352225 0.373441)
+      (xy 10.272216 0.221137) (xy 10.996533 -0.263543) (xy 11.43596 -0.997705) (xy 11.501284 -1.898455)
+      (xy 11.260191 -2.616054) (xy 10.611215 -3.35631) (xy 9.718363 -3.71213) (xy 8.73298 -3.650952)
+      (xy 8.024733 -3.312154) (xy 7.570206 -3.062173) (xy 7.272518 -3.16596) (xy 7.149333 -3.300564)
+      (xy 6.955521 -3.746907) (xy 7.218993 -4.119671) (xy 7.972329 -4.457271) (xy 8.187669 -4.524858)
+      (xy 9.497499 -4.689501) (xy 10.708189 -4.426531)) (layer B.SilkS) (width 0.01))
+  )
+  (gr_text pcbway.com (at 160.02 62.23) (layer B.SilkS)
+    (effects (font (size 2 2) (thickness 0.4)) (justify mirror))
+  )
+  (gr_text "Sponsored by:" (at 175.26 52.07) (layer B.SilkS)
+    (effects (font (size 1.5 1.5) (thickness 0.3)) (justify mirror))
+  )
   (gr_text "Circuit Diagram" (at 123.19 90.17) (layer B.SilkS)
